File: kicad/TP1/TP1.kicad_sch (KiCad schematic)
At the start: 18 parts, among them P1 CONN_20X2, P2 CONN_20X2, U1 MPU-6050, U2 CR2013-MI2120, U4 LM386

Commit message: Actualizacion de KiCad
Connections:
- net +3.3V: now also P1.1 (P1); no longer P2.1 (P1)
- net GPIO_1: now also U2.2 (T_IRQ); no longer U2.5 (T_CS)
- net GPIO_3: now also U2.5 (T_CS); no longer U2.2 (T_IRQ)
- net GPIO_5: now reaches P2.36 (P36)
- net GPIO_5: now also U2.11 (D/~{C})
- net GPIO_7: now reaches P2.38 (P38)
- net GPIO_7: now also U2.12 (RESET)
- net GPIO_8: now reaches P2.40 (P40)
- net GPIO_8: now also U2.13 (~{CS})
- net GPIO_0: no longer names the net of P2.29 (P29)
- net GPIO_0: no longer U2.11 (D/~{C})
- net GPIO_2: no longer names the net of P2.31 (P31)
- net GPIO_2: no longer U2.12 (RESET)
- net GPIO_4: no longer names the net of P2.33 (P33)
- net GPIO_4: no longer U2.13 (~{CS})
- net GPIO_6: no longer names the net of P2.35 (P35)
- no-connect marks 76 -> 77

Commit message: Actualizacion Kicad
Parts:
- C1: footprint Capacitor_THT:C_Disc_D5.0mm_W2.5mm_P5.00mm -> Capacitor_THT:CP_Radial_D8.0mm_P5.00mm; symbol Device:C -> Device:C_Polarized
Changed lines of the file:
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@@
 	)
 	(symbol
-		(lib_id "Device:C")
+		(lib_id "Device:C_Polarized")
 		(at 245.11 58.42 90)
 		(unit 1)
@@
 			)
 		)
-		(property "Footprint" "Capacitor_THT:C_Disc_D5.0mm_W2.5mm_P5.00mm"
+		(property "Footprint" "Capacitor_THT:CP_Radial_D8.0mm_P5.00mm"
 			(at 248.92 57.4548 0)
 			(effects
@@
 			)
 		)
-		(property "Description" "Unpolarized capacitor"
+		(property "Description" "Polarized capacitor"
 			(at 245.11 58.42 0)
 			(effects

Commit message: Correcciones del CAD
Connections:
- net SPI_MOSI: now also U2.10 (SDI(MOSI)); no longer U2.7 (SDO(MISO))
Changed lines of the file:
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@@
 	(title_block
 		(title "GENERATOR Esquemático")
-		(date "31/10/2024")
-		(rev "1.2")
+		(date "10/02/2024")
+		(rev "1.3")
 	)
 	(junction
@@
 	)
 	(no_connect
-		(at 66.04 116.84)
+		(at 66.04 109.22)
 	)
 	(no_connect
@@
 	(wire
 		(pts
+			(xy 66.04 116.84) (xy 68.58 116.84)
+		)
+		(stroke
+			(width 0)
+			(type default)
+		)
+	)
+	(wire
+		(pts
 			(xy 252.73 60.96) (xy 252.73 63.5)
 		)
@@
 		(pts
 			(xy 220.98 39.37) (xy 220.98 40.64)
-		)
-		(stroke
-			(width 0)
-			(type default)
-		)
-	)
-	(wire
-		(pts
-			(xy 66.04 109.22) (xy 68.58 109.22)
 		)
 		(stroke
@@
 	(global_label "SPI_MOSI"
 		(shape input)
-		(at 68.58 109.22 0)
+		(at 68.58 116.84 0)
 		(fields_autoplaced yes)
 		(effects
@@
 		)
 		(property "Intersheetrefs" "${INTERSHEET_REFS}"
-			(at 80.2133 109.22 0)
-			(effects
-				(font
+			(at 80.2133 116.84 0)
+			(effects
+				(font
